Commit message: Enhance dashboard with 4 matplotlib windows and improve URDF structure

File: urdf/robot_model.urdf (robot description, URDF)
Before this commit: robot robot_model, 3 links, 2 joints
Links:
- added link world
- link base_link: mass None -> 5.0; geometry collision box size=0.5 0.5 0.1; visual box size=0.5 0.5 0.1
- link buse_link: mass None -> 0.5; geometry collision cylinder length=0.2 radius=0.05; visual cylinder length=0.2 radius=0.05
- link pyrometer_link: mass None -> 0.1; geometry collision cylinder length=0.1 radius=0.02; visual cylinder length=0.1 radius=0.02
Joints:
- added joint base_to_world: type fixed, parent world, child base_link, origin xyz=0 0 0 rpy=0 0 0
- joint buse_joint: origin xyz=-0.2 0 0.05 -> xyz=-0.2 0 0.15 rpy=0 0 0
- joint pyrometer_joint: origin xyz=0.2 0 0.05 -> xyz=0.2 0 0.1 rpy=0 0 0

Commit message: Update URDF to 6-axis Staubli robot model, enhance launch file and README

File: urdf/robot_model.urdf (robot description, URDF)
Before this commit: robot robot_model, 4 links, 3 joints
Links:
- added link link1, mass 5.0; collision cylinder length=0.3 radius=0.08; visual cylinder length=0.3 radius=0.08
- added link link2, mass 4.0; collision box size=0.6 0.1 0.1; visual box size=0.6 0.1 0.1
- added link link3, mass 3.0; collision cylinder length=0.4 radius=0.06; visual cylinder length=0.4 radius=0.06
- added link link4, mass 2.0; collision box size=0.4 0.08 0.08; visual box size=0.4 0.08 0.08
- added link link5, mass 1.5; collision cylinder length=0.3 radius=0.04; visual cylinder length=0.3 radius=0.04
- added link link6, mass 1.0; collision cylinder length=0.2 radius=0.05; visual cylinder length=0.2 radius=0.05
- link base_link: mass 5.0 -> 10.0; geometry collision cylinder length=0.2 radius=0.1; visual cylinder length=0.2 radius=0.1
- link buse_link: mass 0.5 -> 0.2; geometry collision cylinder length=0.15 radius=0.03; visual cylinder length=0.15 radius=0.03
Joints:
- added joint joint1: type revolute, parent base_link, child link1, origin xyz=0 0 0.2 rpy=0 0 0, axis 0 0 1, limit lower=-3.14159 upper=3.14159 effort=100 velocity=1.0
- added joint joint2: type revolute, parent link1, child link2, origin xyz=0 0 0.3 rpy=1.5708 0 0, axis 0 0 1, limit lower=-2.0944 upper=2.0944 effort=100 velocity=1.0
- added joint joint3: type revolute, parent link2, child link3, origin xyz=0.6 0 0 rpy=0 0 0, axis 0 0 1, limit lower=-2.618 upper=2.618 effort=100 velocity=1.0
- added joint joint4: type revolute, parent link3, child link4, origin xyz=0 0 0.4 rpy=1.5708 0 0, axis 0 0 1, limit lower=-3.14159 upper=3.14159 effort=100 velocity=1.0
- added joint joint5: type revolute, parent link4, child link5, origin xyz=0.4 0 0 rpy=-1.5708 0 0, axis 0 0 1, limit lower=-2.0944 upper=2.0944 effort=100 velocity=1.0
- added joint joint6: type revolute, parent link5, child link6, origin xyz=0 0 0.3 rpy=1.5708 0 0, axis 0 0 1, limit lower=-3.14159 upper=3.14159 effort=100 velocity=1.0
- joint buse_joint: origin xyz=-0.2 0 0.15 rpy=0 0 0 -> xyz=-0.1 0 0.1 rpy=0 0 0; parent base_link -> link6
- joint pyrometer_joint: origin xyz=0.2 0 0.1 rpy=0 0 0 -> xyz=0.1 0 0.1 rpy=0 0 0; parent base_link -> link6

Commit message: ro

File: urdf/robot_model.urdf (robot description, URDF)
Before this commit: robot staubli_tx60, 10 links, 9 joints
Links:
- removed link buse_link
- removed link pyrometer_link
Joints:
- removed joint buse_joint
- removed joint pyrometer_joint
